File: KiCad/canned-ercf-board.kicad_pcb (KiCad board)
At the start: 2 copper layers, 90.8 x 35.6 mm, 33 parts, among them J1 Conn_01x04_Male, J2 Screw_Terminal_01x02, J3 Conn_01x03_Male, J4 Conn_01x03_Male, J5 Conn_01x03_Male, J6 Conn_01x03_Male, J7 Conn_01x04_Male, J8 Conn_01x04_Male, U1 Switching_Regulator_LMP78_05-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, U2 TMC2209_SILENTSTEPSTICK, U3 TMC2209_SILENTSTEPSTICK

Commit message: v1.0-beta2
Parts:
- added C5: 2n2, Capacitor_SMD:C_0603_1608Metric, F.Cu at (80.1, 132.8)
- added C6: 2n2, Capacitor_SMD:C_0603_1608Metric, F.Cu at (88.4, 132.8)
- added C7: 100uF, Capacitor_SMD:CP_Elec_6.3x7.7, F.Cu at (152.9, 126.1)
- added C8: 100uF, Capacitor_SMD:CP_Elec_6.3x7.7, F.Cu at (131.8, 126.2)
- added D4: Yellow, LED_SMD:LED_0603_1608Metric, F.Cu at (158.1, 110.5)
- added D5: Green, LED_SMD:LED_0603_1608Metric, F.Cu at (154.8, 110.5)
- added J9: Conn_01x02, Connector_Molex:Molex_KK-254_AE-6410-02A_1x02_P2.54mm_Vertical, F.Cu at (80.3, 120.7)
- added R10: 10K, Resistor_SMD:R_0603_1608Metric, F.Cu at (91.7, 132.8)
- added R11: 27K, Resistor_SMD:R_0603_1608Metric, F.Cu at (93.4, 132.8)
- added R12: 27K, Resistor_SMD:R_0603_1608Metric, F.Cu at (83.4, 132.8)
- added R13: 27K, Resistor_SMD:R_0603_1608Metric, F.Cu at (85.1, 132.8)
- added R14: 1k, Resistor_SMD:R_0603_1608Metric, F.Cu at (91.9, 122.1)
- added R15: 4K7, Resistor_SMD:R_0603_1608Metric, F.Cu at (135.4, 121.6)
- added R16: 10k, Resistor_SMD:R_0603_1608Metric, F.Cu at (160.4, 121.9)
- added R17: 10k, Resistor_SMD:R_0603_1608Metric, F.Cu at (138.8, 121.6)
- added R8: 10K, Resistor_SMD:R_0603_1608Metric, F.Cu at (86.7, 132.8)
- added R9: 10K, Resistor_SMD:R_0603_1608Metric, F.Cu at (81.8, 132.8)
- C1: value 10uF -> 0u01; footprint Capacitor_SMD:C_0805_2012Metric -> Capacitor_SMD:C_0603_1608Metric
- C2: value 22uF -> 10uF
- C3: value 100uF -> 22uF; footprint Capacitor_SMD:CP_Elec_6.3x7.7 -> Capacitor_SMD:C_0805_2012Metric
- C4: value 100uF -> 2n2; footprint Capacitor_SMD:CP_Elec_6.3x7.7 -> Capacitor_SMD:C_0603_1608Metric
- D1: value Blue -> BAT54C; footprint LED_SMD:LED_0603_1608Metric -> Package_TO_SOT_SMD:SOT-23
- D2: value Yellow -> BAT54C; footprint LED_SMD:LED_0603_1608Metric -> Package_TO_SOT_SMD:SOT-23
- D3: value Green -> Blue
- J1: value Conn_01x04_Male -> Conn_01x02; footprint Connector_Molex:Molex_KK-254_AE-6410-04A_1x04_P2.54mm_Vertical -> Connector_Molex:Molex_KK-254_AE-6410-02A_1x02_P2.54mm_Vertical
- J2: value Screw_Terminal_01x02 -> Conn_01x03_Male; footprint canned-ercf-board:TerminalBlock_bornier-2_P5.08mm_2 -> Connector_Molex:Molex_KK-254_AE-6410-03A_1x03_P2.54mm_Vertical
- J6: value Conn_01x03_Male -> Screw_Terminal_01x02; footprint Connector_Molex:Molex_KK-254_AE-6410-03A_1x03_P2.54mm_Vertical -> canned-ercf-board:TerminalBlock_bornier-2_P5.08mm_2
- R1: value 1k -> 470R
- R2: value 120R -> 47K
- R3: value 10k -> 4K7
- R4: value 10k -> 120R
- moved D1 70.3 mm to (83.4, 136.5), turned to -90 degrees
- moved D2 69.1 mm to (91.1, 136.5), turned to -90 degrees
- moved C4 63.6 mm to (90.1, 132.8), turned to 90 degrees
- moved R2 56.9 mm to (142.4, 110.5)
- moved R4 54.4 mm to (85.0, 116.5), turned to -90 degrees
- moved J6 38.2 mm to (135.1, 112.3), turned to 180 degrees
- moved J2 29.1 mm to (105.9, 119.3), turned to 0 degrees
- moved R3 19.9 mm to (144.1, 110.5), turned to -90 degrees
- moved C1 17.3 mm to (140.6, 110.5), turned to -90 degrees
- moved C3 16.8 mm to (124.8, 110.5), turned to -90 degrees
- moved J3 9.02 mm to (97.0, 119.3)
- moved J4 7.79 mm to (97.0, 111.5)
- moved J1 5.51 mm to (80.2, 114.0)
- moved R1 4.44 mm to (95.0, 132.8), turned to -90 degrees
- moved R5 4.19 mm to (145.9, 110.5)
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Connections:
- net DIAG_0 renamed DRIVER_0_DIAG
- net DIAG_1 renamed DRIVER_1_DIAG
- net DIR_0 renamed DRIVER_0_DIR
- net DIR_1 renamed DRIVER_1_DIR
- net STEP_0 renamed DRIVER_0_STEP
- net STEP_1 renamed DRIVER_1_STEP
- A1 pad 1: EXTRA -> IO_2
- A1 pad 2: unconnected-(A1-Pad2) -> VIN_MON
- A1 pad 24: ENDSTOP -> IO_1
- A1 pad 25: DRIVES_UART -> DRIVER_RX
- A1 pad 27: TX -> DRIVER_TX
- A1 pad 5: SERVO -> Net-(A1-Pad5)
- A1 pad 6: ENCODER -> IO_3
- C1 pad 1: VDC -> VIN_MON
- C2 pad 1: +5V -> VDC
- C3 pad 1: VDC -> +5V
- C4 pad 1: VDC -> IO_3
- D1 pad 1: Net-(D1-Pad1) -> IO_1
- D1 pad 2: VDC -> IO_2
- D2 pad 1: Net-(D2-Pad1) -> IO_3
- D2 pad 2: +5V -> unconnected-(D2-Pad2)
- D3 pad 2: +3V3 -> VDC
- J1 pad 1: CAN_H -> CAN_L
- J1 pad 2: CAN_L -> CAN_H
- J2 pad 1: GND -> +5V
- J2 pad 2: VDC -> GND
- J3 pad 1: +5V -> +3V3
- J3 pad 3: SERVO -> IO_3_IN
- J4 pad 3: ENCODER -> IO_2_IN
- J5 pad 3: EXTRA -> IO_1_IN
- J6 pad 1: +3V3 -> GND
- J6 pad 2: GND -> VDC
- JP1 pad 1: CAN_H -> CAN_L
- JP2 pad 2: DRIVES_UART -> DRIVER_RX
- JP3 pad 2: DRIVES_UART -> DRIVER_RX
- R1 pad 1: DRIVES_UART -> IO_0_OUT
- R1 pad 2: TX -> Net-(A1-Pad5)
- R2 pad 1: CAN_L -> VDC
- R2 pad 2: Net-(JP1-Pad2) -> VIN_MON
- R3 pad 1: DRIVES_EN -> VIN_MON
- R3 pad 2: +3V3 -> GND
- R4 pad 1: DRIVES_EN -> CAN_H
- R4 pad 2: +3V3 -> Net-(JP1-Pad2)
- R5 pad 1: Net-(D1-Pad1) -> Net-(D3-Pad1)
- R6 pad 1: Net-(D2-Pad1) -> Net-(D4-Pad1)
- R7 pad 1: Net-(D3-Pad1) -> Net-(D5-Pad1)
- U2 pad JP1_4: Net-(JP2-Pad1) -> Net-(JP2-Pad3)
- U2 pad JP1_5: Net-(JP2-Pad3) -> Net-(JP2-Pad1)
- U3 pad JP1_4: Net-(JP3-Pad1) -> Net-(JP3-Pad3)
- U3 pad JP1_5: Net-(JP3-Pad3) -> Net-(JP3-Pad1)
Routing:
- net +3V3: track 140.8 -> 239.6 mm, vias 0 -> 1
- net VIN_MON: track 0.00 -> 78.5 mm
- net DRIVES_UART: track 77.3 -> 0.00 mm, vias 1 -> 0
- net DRIVER_RX: track 0.00 -> 77.2 mm, vias 0 -> 3
- net Net-(D3-Pad1): track 67.6 -> 6.43 mm
- net EXTRA: track 56.2 -> 0.00 mm
- net IO_1_IN: track 0.00 -> 38.0 mm
- net IO_2_IN: track 0.00 -> 36.1 mm
- net SERVO: track 32.1 -> 0.00 mm
- net ENCODER: track 25.0 -> 0.00 mm
- net IO_1: track 0.00 -> 22.9 mm
- net IO_0_OUT: track 0.00 -> 22.1 mm
- net ENDSTOP: track 20.6 -> 0.00 mm
- net IO_3_IN: track 0.00 -> 19.7 mm
- net Net-(D5-Pad1): track 0.00 -> 17.4 mm
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Other:
- board text added: ".out"
- board text added: "DRIVER_0"
- board text added: "DRIVER_1"
- board text added: "IO_0"
- board text added: "IO_1"
- board text added: "IO_2"
- board text added: "IO_3"
- board text added: "io0"
- board text added: "io1.in"
- board text added: "io2.in"
- board text added: "io3.in"
- board text added: "v1.0-beta2"
- board text removed: "ENC"
- board text removed: "END"
- board text removed: "EXTRA"
- board text removed: "GEAR"
- board text removed: "PA02"
- board text removed: "PA04"
- board text removed: "PA05"
- board text removed: "PA19"
- board text removed: "SELECTOR"
- board text removed: "SERVO"
- board text removed: "v1.0-beta1"
