File: KiCad/canned-ercf-board.kicad_sch (KiCad schematic)
At the start: 33 parts, among them J1 Conn_01x04_Male, J2 Screw_Terminal_01x02, J3 Conn_01x03_Male, J4 Conn_01x03_Male, J5 Conn_01x03_Male, J6 Conn_01x03_Male, J7 Conn_01x04_Male, J8 Conn_01x04_Male, U1 Switching_Regulator_LMP78_05-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, U2 TMC2209_SILENTSTEPSTICK, U3 TMC2209_SILENTSTEPSTICK

Commit message: v1.0-beta2
Parts:
- removed A1: Sammy_C21, canned-ercf-board:Sammy_C21_Module_DIL32_2.54, symbol canned-ercf-board:Sammy_C21
- removed C1: 10uF, Capacitor_SMD:C_0805_2012Metric, symbol Device:C_Small
- removed C2: 22uF, Capacitor_SMD:C_0805_2012Metric, symbol Device:C_Small
- removed C3, C4: 100uF, Capacitor_SMD:CP_Elec_6.3x7.7, symbol Device:C_Polarized_Small_US
- removed D1: Blue, LED_SMD:LED_0603_1608Metric, symbol Device:LED_Small
- removed D2: Yellow, LED_SMD:LED_0603_1608Metric, symbol Device:LED_Small
- removed D3: Green, LED_SMD:LED_0603_1608Metric, symbol Device:LED_Small
- removed J1: Conn_01x04_Male, Connector_Molex:Molex_KK-254_AE-6410-04A_1x04_P2.54mm_Vertical, symbol Connector_Generic:Conn_01x04
- removed J2: Screw_Terminal_01x02, canned-ercf-board:TerminalBlock_bornier-2_P5.08mm_2, symbol Connector:Screw_Terminal_01x02
- removed J3, J4, J5, J6: Conn_01x03_Male, Connector_Molex:Molex_KK-254_AE-6410-03A_1x03_P2.54mm_Vertical, symbol Connector_Generic:Conn_01x03
- removed J7, J8: Conn_01x04_Male, Connector_Molex:Molex_KK-254_AE-6410-04A_1x04_P2.54mm_Vertical, symbol Connector:Conn_01x04_Male
- removed JP1: SolderJumper_2_Open, Jumper:SolderJumper-2_P1.3mm_Open_TrianglePad1.0x1.5mm, symbol Jumper:SolderJumper_2_Open
- removed JP2, JP3: SolderJumper_3_Bridged12, Jumper:SolderJumper-3_P1.3mm_Bridged12_RoundedPad1.0x1.5mm, symbol Jumper:SolderJumper_3_Bridged12
- removed R1: 1k, Resistor_SMD:R_0603_1608Metric, symbol Device:R_Small
- removed R2, R7: 120R, Resistor_SMD:R_0603_1608Metric, symbol Device:R_Small
- removed R3, R4: 10k, Resistor_SMD:R_0603_1608Metric, symbol Device:R
- removed R5: 4K7, Resistor_SMD:R_0603_1608Metric, symbol Device:R_Small
- removed R6: 390R, Resistor_SMD:R_0603_1608Metric, symbol Device:R_Small
- removed U1: Switching_Regulator_LMP78_05-1.5, canned-ercf-board:Switching_regulator_POL_LMP78_1.5, symbol canned-ercf-board:Switching_Regulator_LMP78_05-1.5
- removed U2, U3: TMC2209_SILENTSTEPSTICK, MODULE_TMC2208_SILENTSTEPSTICK, symbol canned-ercf-board:TMC2209_SILENTSTEPSTICK
Connections:
- no-connect marks 18 -> 0
Other:
- added sheet Drivers (drivers.kicad_sch)
- added sheet Input_output (input_output.kicad_sch)
- added sheet MCU (mcu.kicad_sch)
- note added: "Drivers"
- note added: "In-/Output"
- note removed: "- ENCODER"
- note removed: "- EXTRA (TOOLHEAD)"
- note removed: "- SELECTOR ENDSTOP"
- note removed: "- SERVO"
- note removed: "CAN"
- note removed: "DCDC-5V"
- note removed: "ENDSTOPS"
- note removed: "GEAR STEPPER"
- note removed: "SELECTOR STEPPER"
- moved on the sheet: H1, H2, H3
